File: frontend/frontend.kicad_sch (KiCad schematic)
At the start: 59 parts, among them J1 REF_IN, J2 REF_S_P, J3 REF_S_N, J4 REF_GND, U1 ADG722, U2 ADG722, U3 OPA2387DGKT, U4 LM358, U5 LTC2508CDKD-32, U6 ADG722, U8 74HC595

Commit message: 7
Parts:
- added C17, C38, C39, C40, C41: 100n, Capacitor_SMD:C_0805_2012Metric_Pad1.18x1.45mm_HandSolder, symbol Device:C
- added F1: ВП2Б-1В, 1.25A, Passives:KLS5-266(FH-100), symbol Passives:KLS5-266(FH-100)
- added R37: 0,005, Resistor_SMD:R_2512_6332Metric, symbol Device:R
- added R38: 24k, Resistor_SMD:R_1206_3216Metric_Pad1.30x1.75mm_HandSolder, symbol Device:R
- added R39: 750, Resistor_SMD:R_1206_3216Metric_Pad1.30x1.75mm_HandSolder, symbol Device:R
- added R40: 10, Resistor_SMD:R_1206_3216Metric_Pad1.30x1.75mm_HandSolder, symbol Device:R
- added U12: MAX4208, Package_SO:MSOP-8_3x3mm_P0.65mm, symbol New_Library1:MAX4208
- R10: value 4k7 -> 6k2
- R11: value 4k7 -> 2k7
- R12: value 13k -> 10k
- R34: value 47 -> 10
Connections:
- net +5V: now also C39.1, U12.8 (VDD)
- net -0.6V: now also C40.1, U12.1 (MODE), U12.4 (VSS)
- net -5V: now also C17.1, C38.1; no longer C30.2, C31.2
- net GND: now also C30.2, C31.2, C17.2, C38.2, C39.2, C40.2, C41.2
- net at R3.1, RV3.2: now also R37.1, U12.2 (IN-)
- net +2V: no longer names the net of U3.6 (-), U3.7
- net +2V: now also R40.2; no longer R11.2, U6.6 (D2)
- new net: R38.1, R39.2, U12.6 (FB)
- new net: F1.2, R37.2, U12.3 (IN+)
- new net: R38.2, U12.7 (OUT)
- new net +1V65: C41.1, R11.2, R39.1, R40.1, U12.5 (REF), U6.6 (D2)
Other:
- note added: "G=3.3"
- note added: "G=33"
- moved on the sheet: C27, C28, C29, C30, R32, R33, U1C, U2C, U6C

Commit message: 7
Parts:
- removed R34, R40: 10, Resistor_SMD:R_1206_3216Metric_Pad1.30x1.75mm_HandSolder, symbol Device:R
- added C42, C43, C44, C47, C48, C49, C50: 10n, Capacitor_SMD:C_0805_2012Metric_Pad1.18x1.45mm_HandSolder, symbol Device:C
- added C45, C46, C52: 100n, Capacitor_SMD:C_0805_2012Metric_Pad1.18x1.45mm_HandSolder, symbol Device:C
- added C51: 47u, Capacitor_SMD:C_0805_2012Metric_Pad1.18x1.45mm_HandSolder, symbol Device:C
- added D2, D3, D4, D5, D6, D7: 1N4148W, Diode_SMD:D_SOD-123, symbol Diode:1N4148W
- added D8, D9: CUS520, Diode_SMD:D_SOD-323, symbol Device:D_Schottky
- added F2: 0.3A, Passives:KLS5-266(FH-100), symbol Passives:KLS5-266(FH-100)
- added K1, K2: NRP26-A05D, Relay_THT:Relay_StandexMeder_DIP_LowProfile, symbol Relay:DIPxx-1Axx-11x
- added Q2, Q3: MMBT2222A, Package_TO_SOT_SMD:SOT-23, symbol Transistor_BJT:MMBT2222A
- added R41: 0.5 HoJLR2512-3W-500mR-1%, Resistor_SMD:R_2512_6332Metric, symbol Device:R
- added R42, R43, R46, R47, R50, R51: 1k, Resistor_SMD:R_1206_3216Metric_Pad1.30x1.75mm_HandSolder, symbol Device:R
- added R44: 10 PRG3216P-10R0-D-T5, Resistor_SMD:R_2512_6332Metric, symbol Device:R
- added R48, R53: 68k, Resistor_SMD:R_1206_3216Metric_Pad1.30x1.75mm_HandSolder, symbol Device:R
- added R49, R52, R54, R55: 4k7, Resistor_SMD:R_1206_3216Metric_Pad1.30x1.75mm_HandSolder, symbol Device:R
- added R56: 33, Resistor_SMD:R_1206_3216Metric_Pad1.30x1.75mm_HandSolder, symbol Device:R
- added R57: 10k, Resistor_SMD:R_1206_3216Metric_Pad1.30x1.75mm_HandSolder, symbol Device:R
- added U13: OPA2186DR, Package_SO:VSSOP-8_3x3mm_P0.65mm, symbol Amplifier_Operational:OPA2325
- added U14: ADG722, Library:uSOIC, symbol New_Library:ADG722
- C32: value 1u -> 4u7
- F1: value ВП2Б-1В, 1.25A -> 10A
- R1: value 3k -> 1k
- R19, R20: value 47 -> 10
- R37: value 0,005 -> 0,01 RLP25FEGR010
- R38: value 24k -> 68k
- R39: value 750 -> 4k7
- RV1, RV2, RV3: value Varistor -> KSE-14K391
- TH1: value 3k -> 1k; footprint Resistor_THT:R_Axial_Power_L20.0mm_W6.4mm_P5.08mm_Vertical -> Resistor_THT:R_Axial_Power_L20.0mm_W6.4mm_P7.62mm_Vertical
- U3: value OPA2387DGKT -> OPA2186DR; footprint Package_SO:SOIC-8_3.9x4.9mm_P1.27mm -> Package_SO:VSSOP-8_3x3mm_P0.65mm
Connections:
- net +1V65: now also U3.6 (-), U3.7, R49.1, R52.1
- net +2V5: now also C33.1, C34.1, U5.3 (V_{DD})
- net +3V3: now also D8.1 (K)
- net +5V: now also C45.1, C52.1, R56.1, U13.8 (V+), U14.8 (VDD)
- net -5V: now also C46.1, U13.4 (V-)
- net ADC_IN+: now also R19.2, U6.2 (D1), U6.5 (S2), U14.2 (D1), U14.6 (D2); no longer C9.1, R21.2, U6.1 (S1)
- net GND: now also C45.2, C46.2, C51.2, D9.2 (A), Q2.2 (E), Q3.2 (E), R57.2
- net at R3.1, R37.1, RV3.2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: now also C43.2, C47.2, C49.2, D2.1 (K), D3.2 (A), D4.1 (K), D5.2 (A), D6.1 (K), D7.2 (A), R41.1, R44.1
- net SW_LOW: now reaches C27.2, C28.2, C29.2, R32.2, R33.2, U1.4 (GND), U2.4 (GND), U6.4 (GND)
- net SW_LOW: now also C52.2, U14.4 (GND)
- net at R10.1, R21.1, U3.1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: now also C44.2
- net at R10.2, R11.1, U3.2 (-): now also C44.1
- net at C6.1, C7.2, R19.1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: now also D8.2 (A), D9.1 (K)
- net at R38.1, R39.2, U12.6 (FB): now also C42.2
- net at F1.2, R37.2: now also R42.2; no longer U12.3 (IN+)
- net CURR_10A: now reaches R38.2, U12.7 (OUT)
- net CURR_10A: now also C42.1
- net RANGE10 renamed SW_RANGE10
- net RANGE100 renamed SW_RANGE100
- net RANGE1000 renamed SW_RANGE1000
- net SW_ADC_2V renamed SW_1V65_IN
- net SW_ADC_IN renamed SW_VOLTS_IN
- new net: C47.1, D4.2 (A), D5.1 (K), R47.1, U13.3 (+)
- new net: K1.1, K1.14, R41.2, R50.2
- new net: K1.2, Q2.3 (C), R54.1
- new net: C51.1, K1.6, K2.6, R56.2
- new net: F2.2, K1.7, K1.8, K2.7, K2.8
- new net: R55.1, R57.1
- new net: R50.1, R51.2
- new net: Q2.1 (B), R55.2
- new net: C48.1, R48.1, R49.2, U13.2 (-)
- new net: C49.1, D6.2 (A), D7.1 (K), R51.1, U13.5 (+)
- new net: C50.1, R52.2, R53.1, U13.6 (-)
- new net: R42.1, R43.2
- new net: C43.1, D2.2 (A), D3.1 (K), R43.1, U12.3 (IN+)
- new net: R46.1, R47.2
- new net: K2.1, K2.14, R44.2, R46.2
- new net: Q3.1 (B), R54.2
- new net: K2.2, Q3.3 (C)
- new net CURR_10mA: C48.2, R48.2, U13.1, U14.1 (S1)
- new net CURR_200mA: C50.2, R53.2, U13.7, U14.5 (S2)
- new net SW_CURR_10mA: U14.7 (IN1)
- new net SW_CURR_200mA: U14.3 (IN2)
- new net VOLTS: C9.1, R21.2, U6.1 (S1)
Other:
- note added: "0.1V/0.01A"
- note added: "0.1V/0.2A"
- note added: "0.1V/10A"
- note added: "G=15.5"
- note removed: "G=33"
- moved on the sheet: C1, C10, C17, C2, C27, C28, C29, C3, C30, C31, C32, C33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

Commit message: 8
Parts:
- added C53: 100n, Capacitor_SMD:C_0805_2012Metric_Pad1.18x1.45mm_HandSolder, symbol Device:C
- added R34, R40, R45, R58, R59, R60: 10k, Resistor_THT:R_Axial_DIN0207_L6.3mm_D2.5mm_P15.24mm_Horizontal, symbol Device:R
- added R61: 10, Resistor_THT:R_Axial_DIN0207_L6.3mm_D2.5mm_P15.24mm_Horizontal, symbol Device:R
- added U15: 74HC595, Package_SO:SOIC-16_3.9x9.9mm_P1.27mm, symbol 74xx:74HC595
Connections:
- net +3V3: now also R34.1, R60.1, R61.1, U15.10 (~{SRCLR})
- net +5V: now also R45.2, R58.2, R59.2
- net GND: now also C53.2, R40.1, U15.8 (GND)
- net SW_1V65_IN: now also R40.2
- net SW_CURR_10mA: now also R59.1, U15.15 (QA)
- net SW_CURR_200mA: now also R58.1, U15.1 (QB)
- net SW_VOLTS_IN: now also R45.1
- net SW_CURR_RANGE: now reaches R55.1, R57.1
- net SW_CURR_RANGE: now also U8.7 (QH)
- net at U8.11 (SRCLK): now also U15.11 (SRCLK)
- net at U8.12 (RCLK): now also U15.12 (RCLK)
- net at U8.13 (~{OE}): now also R34.2
- net at U8.9 (QH'): now also U15.14 (SER)
- new net: C53.1, R61.2, U15.16 (VCC)
- new net: R60.2, U15.13 (~{OE})
Other:
- moved on the sheet: C10, R22, U8

Commit message: 9
Parts:
- added C54, C55: 4u7, Capacitor_SMD:C_0805_2012Metric_Pad1.18x1.45mm_HandSolder, symbol Device:C
- added H1, H2, H3, H4: MountingHole, MountingHole:MountingHole_3.2mm_M3, symbol Mechanical:MountingHole
- added J10: GND, Passives:Conn-1-6x6-OD3mm, symbol Connector:Conn_01x01_Socket
- added J11: Conn_02x13_Odd_Even, Connector_IDC:IDC-Header_2x13_P2.54mm_Vertical, symbol Connector_Generic:Conn_02x13_Odd_Even
- added J12, J13, J14, J15, J16, J17, J18: Conn_01x01_Socket, Connector_PinHeader_2.54mm:PinHeader_1x01_P2.54mm_Vertical, symbol Connector:Conn_01x01_Socket
- added J19: A, Passives:Conn-1-6x6-OD3mm, symbol Connector:Conn_01x01_Socket
- added J5: mA, Passives:Conn-1-6x6-OD3mm, symbol Connector:Conn_01x01_Socket
- added J6: V, Passives:Conn-1-6x6-OD3mm, symbol Connector:Conn_01x01_Socket
- added J7: Common, Passives:Conn-1-6x6-OD3mm, symbol Connector:Conn_01x01_Socket
- added J8: +6V, Passives:Conn-1-6x6-OD3mm, symbol Connector:Conn_01x01_Socket
- added J9: -10V, Passives:Conn-1-6x6-OD3mm, symbol Connector:Conn_01x01_Socket
- added R62, R63: 10, Resistor_SMD:R_1206_3216Metric_Pad1.30x1.75mm_HandSolder, symbol Device:R
- K1, K2: footprint Relay_THT:Relay_StandexMeder_DIP_LowProfile -> Passives:NPR26
- R1: value 1k -> 1k/2W
- R10: value 6k2 -> 6k2/0.1%
- R11: value 2k7 -> 2k7/0.1%
- R12, R13, R6: value 10k -> 10k/0.1%
- R14, R15, R2, R4, R5: value 5M -> 5M/0.1%
- R22, R34, R40, R45, R58, R59, R60, R61: footprint Resistor_THT:R_Axial_DIN0207_L6.3mm_D2.5mm_P15.24mm_Horizontal -> Resistor_SMD:R_1206_3216Metric_Pad1.30x1.75mm_HandSolder
- R37: footprint Resistor_SMD:R_2512_6332Metric -> Passives:2512 Big
- R38, R48, R53: value 68k -> 68k/0.1%
- R39, R49, R52: value 4k7 -> 4k7/0.1%
- R44: footprint Resistor_SMD:R_2512_6332Metric -> Passives:1206 Vertical
- R7: value 100k -> 100k/0.1%
- R8: value 1M -> 1M/0.1%
- R9: value 20meg -> 20meg/0.1%
Connections:
- net +1V65: now also C55.1, R62.2; no longer U3.6 (-), U3.7
- net +2V5: now also R63.1; no longer C33.1, C34.1, U5.3 (V_{DD})
- net +3V3: now also C54.1
- net +6V: now also J8.1 (Pin_1)
- net -10V: now also J9.1 (Pin_1)
- net GND: now also C54.2, C55.2, J10.1 (Pin_1)
- net COMMON: now reaches C43.2, C47.2, C49.2, D2.1 (K), D3.2 (A), D4.1 (K), D5.2 (A), D6.1 (K), D7.2 (A), R3.1, R37.1, R41.1, R44.1, RV3.2, U12.2 (IN-)
- net COMMON: now also J7.1 (Pin_1)
- net SHIFT_SRCLK: now reaches R34.2, U8.13 (~{OE})
- net SHIFT_SRCLK: now also R60.2, U15.11 (SRCLK), U15.13 (~{OE}), U8.11 (SRCLK), J11.23 (Pin_23), J11.26 (Pin_26)
- net SHIFT_RCLK: now reaches U15.12 (RCLK), U8.12 (RCLK)
- net SHIFT_RCLK: now also J11.25 (Pin_25)
- net at U15.2 (QC): now also J12.1 (Pin_1)
- net at U15.3 (QD): now also J13.1 (Pin_1)
- net at U15.4 (QE): now also J14.1 (Pin_1)
- net at U15.5 (QF): now also J15.1 (Pin_1)
- net at U15.6 (QG): now also J16.1 (Pin_1)
- net at U15.7 (QH): now also J17.1 (Pin_1)
- net at U15.9 (QH'): now also J18.1 (Pin_1)
- net V: now reaches R1.1
- net V: now also J6.1 (Pin_1)
- net mA: now reaches F2.1
- net mA: now also J5.1 (Pin_1)
- net A: now reaches F1.1
- net A: now also J19.1 (Pin_1)
- net RDLA: now reaches U5.1 (~{RDLA})
- net RDLA: now also J11.5 (Pin_5)
- net MCLK: now reaches U5.13 (MCLK)
- net MCLK: now also J11.1 (Pin_1)
- net SYNC: now reaches U5.14 (SYNC)
- net SYNC: now also J11.3 (Pin_3)
- net DRL: now reaches U5.15 (~{DRL})
- net DRL: now also J11.9 (Pin_9)
- net SDOA: now reaches U5.17 (SDOA)
- net SDOA: now also J11.15 (Pin_15)
- net SCKA: now reaches U5.18 (SCKA)
- net SCKA: now also J11.13 (Pin_13)
- net SCKB: now reaches U5.19 (SCKB)
- net SCKB: now also J11.17 (Pin_17)
- net RDLB: now reaches U5.2 (~{RDLB})
- net RDLB: now also J11.7 (Pin_7)
- net SDOB: now reaches U5.20 (SDOB)
- net SDOB: now also J11.19 (Pin_19)
- net BUSY: now reaches U5.21 (BUSY)
- net BUSY: now also J11.11 (Pin_11)
- net SHIFT_DATA: now reaches U8.14 (SER)
- net SHIFT_DATA: now also J11.21 (Pin_21)
- new net: C33.1, C34.1, R63.2, U5.3 (V_{DD})
- new net: R62.1, U3.6 (-), U3.7
- new net: J11.10 (Pin_10), J11.12 (Pin_12), J11.14 (Pin_14), J11.16 (Pin_16), J11.18 (Pin_18), J11.2 (Pin_2), J11.20 (Pin_20), J11.22 (Pin_22), J11.24 (Pin_24), J11.4 (Pin_4), J11.6 (Pin_6), J11.8 (Pin_8)
Other:
- moved on the sheet: C2, C3, C4, C5, J1, R16, R17, R18, U2B, U6B

Commit message: 11
Parts:
- removed J12: Conn_01x01_Socket, Connector_PinHeader_2.54mm:PinHeader_1x01_P2.54mm_Vertical, symbol Connector:Conn_01x01_Socket
- added C56, C58, C59: 4u7, Capacitor_SMD:C_0805_2012Metric_Pad1.18x1.45mm_HandSolder, symbol Device:C
- added C57: 100n, Capacitor_SMD:C_0805_2012Metric_Pad1.18x1.45mm_HandSolder, symbol Device:C
- added H5, H6, H7, H8: MountingHole, MountingHole:MountingHole_3.2mm_M3, symbol Mechanical:MountingHole
- added U16: ADG722, Library:uSOIC, symbol New_Library:ADG722
- R14, R15, R2, R4, R5: value 5M/0.1% -> 2M2/0.1%
- R6: value 10k/0.1% -> 5k/0.1%
- R62: value 10 -> 47
- R7: value 100k/0.1% -> 50k/0.1%
- R8: value 1M/0.1% -> 500k/0.1%
- R9: value 20meg/0.1% -> 10meg/0.1%
Connections:
- net +1V65: now also C56.1, C58.1
- net +5V: now also C57.1, U16.8 (VDD)
- net -5V: now also C59.1
- net ADC_IN+: now also U16.2 (D1)
- net CURR_10A: now also U16.1 (S1)
- net GND: now also C56.2, C58.2, C59.2, U16.3 (IN2), U16.5 (S2)
- net SW_LOW: now also C57.2, U16.4 (GND)
- net SW_CURR_10A: now reaches U15.2 (QC)
- net SW_CURR_10A: now also U16.7 (IN1)
Other:
- moved on the sheet: C17, C30, C31, C38, C39, C40, C45, C46, H1, H2, H3, H4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

Commit message: 12
Parts:
- removed R60: 10k, Resistor_SMD:R_1206_3216Metric_Pad1.30x1.75mm_HandSolder, symbol Device:R
- added C60, C61, C62, C63: 1u, Capacitor_SMD:C_0805_2012Metric_Pad1.18x1.45mm_HandSolder, symbol Device:C
Connections:
- net +3V3: now also R45.2, R58.2, R59.2
- net +5V: now also C60.2, C61.2, C62.2; no longer R45.2, R58.2, R59.2
- net -0.6V: now also C61.1
- net -5V: now also C60.1, C62.1, C63.1
- net DRL: now also J11.21 (Pin_21); no longer J11.9 (Pin_9)
- net GND: now also J11.10 (Pin_10), J11.12 (Pin_12), J11.14 (Pin_14), J11.16 (Pin_16), J11.18 (Pin_18), J11.2 (Pin_2), J11.20 (Pin_20), J11.22 (Pin_22), J11.24 (Pin_24), J11.4 (Pin_4), J11.6 (Pin_6), J11.8 (Pin_8), C63.2
- net MCLK: now also J11.25 (Pin_25); no longer J11.1 (Pin_1)
- net RDLA: now also J11.9 (Pin_9); no longer J11.5 (Pin_5)
- net SCKA: now also J11.17 (Pin_17); no longer J11.13 (Pin_13)
- net SCKB: now also J11.15 (Pin_15); no longer J11.17 (Pin_17)
- net SDOA: now also J11.19 (Pin_19); no longer J11.15 (Pin_15)
- net SDOB: now also J11.13 (Pin_13); no longer J11.19 (Pin_19)
- net SEL0: now also U15.2 (QC); no longer U8.3 (QD)
- net SEL1: now also U15.1 (QB); no longer U8.4 (QE)
- net SHIFT_DATA: now also J11.3 (Pin_3); no longer J11.21 (Pin_21)
- net SHIFT_RCLK: now also J11.5 (Pin_5); no longer J11.25 (Pin_25)
- net SHIFT_SRCLK: now also J11.1 (Pin_1); no longer J11.23 (Pin_23), J11.26 (Pin_26)
- net SW_1V65_IN: now also U8.15 (QA); no longer U8.6 (QG)
- net SW_CURR_10A: now also U8.3 (QD); no longer U15.2 (QC)
- net SW_CURR_10mA: now also U8.7 (QH); no longer U15.15 (QA)
- net SW_CURR_200mA: now also U8.2 (QC); no longer U15.1 (QB)
- net SW_CURR_RANGE: now also U8.1 (QB); no longer U8.7 (QH)
- net SW_RANGE10: now also U8.4 (QE); no longer U8.2 (QC)
- net SW_RANGE100: now also U8.6 (QG); no longer U8.1 (QB)
- net SW_RANGE1000: now also U8.5 (QF); no longer U8.15 (QA)
- net SW_VOLTS_IN: now also U15.15 (QA); no longer U8.5 (QF)
- net SYNC: now also J11.23 (Pin_23); no longer J11.3 (Pin_3)
Other:
- moved on the sheet: C31, C38, C39, C40, C45, C46, C59, U12B, U13C, U4C

Commit message: 13
Parts:
- removed C10: 100n, Capacitor_SMD:C_0805_2012Metric_Pad1.18x1.45mm_HandSolder, symbol Device:C
- removed J13, J18: Conn_01x01_Socket, Connector_PinHeader_2.54mm:PinHeader_1x01_P2.54mm_Vertical, symbol Connector:Conn_01x01_Socket
- removed R22: 10, Resistor_SMD:R_1206_3216Metric_Pad1.30x1.75mm_HandSolder, symbol Device:R
- removed R34: 10k, Resistor_SMD:R_1206_3216Metric_Pad1.30x1.75mm_HandSolder, symbol Device:R
- removed U15, U8: 74HC595, Package_SO:SOIC-16_3.9x9.9mm_P1.27mm, symbol 74xx:74HC595
- added J12: Conn_01x01_Socket, Connector_PinHeader_2.54mm:PinHeader_1x01_P2.54mm_Vertical, symbol Connector:Conn_01x01_Socket
- added U8: TCA9535DBR, Package_SO:SSOP-24_5.3x8.2mm_P0.65mm, symbol Interface_Expansion:TCA9535DBR
Connections:
- net GND: now also J11.26 (Pin_26), U8.12 (GND), U8.2 (A1), U8.21 (A0), U8.3 (A2)
- net SEL0: now also U8.14 (P11)
- net SEL1: now also U8.15 (P12)
- net SW_1V65_IN: now also U8.13 (P10)
- net SW_CURR_10A: now also U8.7 (P03)
- net SW_CURR_10mA: now also U8.11 (P07)
- net SW_CURR_200mA: now also U8.6 (P02)
- net SW_CURR_RANGE: now also U8.5 (P01)
- net SW_RANGE10: now also U8.8 (P04)
- net SW_RANGE100: now also U8.10 (P06)
- net SW_RANGE1000: now also U8.9 (P05)
- net SW_VOLTS_IN: now also U8.16 (P13)
- net at C53.1, R61.2: now also U8.24 (VCC)
- net at J14.1 (Pin_1): now also U8.17 (P14)
- net at J16.1 (Pin_1): now also U8.19 (P16)
- net at J17.1 (Pin_1): now also U8.20 (P17)
- net at J15.1 (Pin_1): now also U8.18 (P15)
- net SHIFT_DATA renamed SCL
- net SCL: now also U8.22 (SCL)
- net SHIFT_RCLK: no longer names the net of J11.5 (Pin_5)
- net SHIFT_SRCLK renamed SDA
- net SDA: now also U8.23 (SDA)
- new net: J12.1 (Pin_1), U8.4 (P00)
Other:
- moved on the sheet: C53, J14, J15, J16, J17, R61
