File: frontend/Power.kicad_sch (KiCad schematic)
At the start: 34 parts, among them Q1 BD136, U10 UA723, U11 NCP161, U7 XC6206P252MR, U9 XC6206P332MR

Commit message: 9
Connections:
- net +2V5: now also C37.1, U7.2 (VO)
Changed lines of the file:
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@@
+	)
+	(junction
+		(at 189.23 82.55)
+		(diameter 0)
+		(color 0 0 0 0)
 	)
 	(junction
@@
 		(pts
 			(xy 54.61 38.1) (xy 66.04 38.1)
+		)
+		(stroke
+			(width 0)
+			(type default)
+		)
+	)
+	(wire
+		(pts
+			(xy 189.23 81.28) (xy 189.23 82.55)
 		)
 		(stroke
@@
 					(unit 1)
 				)
+			)
+		)
+	)
+	(symbol
+		(lib_id "power:+2V5")
+		(at 189.23 81.28 0)
+		(unit 1)
+		(exclude_from_sim no)
+		(in_bom yes)
+		(on_board yes)
+		(dnp no)
+		(fields_autoplaced yes)
+		(property "Reference" "#PWR0122"
+			(at 189.23 85.09 0)
+			(effects
+				(font
+					(size 1.27 1.27)
+				)
+				(hide yes)
+			)
+		)
+		(property "Value" "+2V5"
+			(at 189.23 76.2 0)
+			(effects
+				(font
+					(size 1.27 1.27)
+				)
+			)
+		)
+		(property "Footprint" ""
+			(at 189.23 81.28 0)
+			(effects
+				(font
+					(size 1.27 1.27)
+				)
+				(hide yes)
+			)
+		)
+		(property "Datasheet" ""
+			(at 189.23 81.28 0)
+			(effects
+				(font
+					(size 1.27 1.27)
+				)
+				(hide yes)
+			)
+		)
+		(property "Description" "Power symbol creates a global label with name \"+2V5\""
+			(at 189.23 81.28 0)
+			(effects
+				(font
+					(size 1.27 1.27)
+				)
+				(hide yes)
+			)
+		)
+		(pin "1"
+		)
+		(instances
+			(project "frontend"
+				(path "/ab777daf-a678-4c7c-8aaf-8ba908a1ed49/3bd9bcdd-eb84-44eb-88c5-a95914037641"
+					(reference "#PWR0122")
+					(unit 1)
+				)

Commit message: 12
Parts:
- U11: value NCP161 -> NCP161ASN500T1G
Changed lines of the file:
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@@
 			)
 		)
-		(property "Value" "NCP161"
+		(property "Value" "NCP161ASN500T1G"
 			(at 169.545 35.56 0)
 			(effects
