File: frontend/Power.kicad_sch (KiCad schematic)
At the start: 34 parts, among them Q1 BD136, U10 UA723, U11 NCP161ASN500T1G, U7 XC6206P252MR, U9 XC6206P332MR

Commit message: 13
Parts:
- added TP1: -0.6V, Connector_Pin:Pin_D1.3mm_L11.3mm_W2.8mm_Flat, symbol Connector:TestPoint
- added TP2: -5V, Connector_Pin:Pin_D1.3mm_L11.3mm_W2.8mm_Flat, symbol Connector:TestPoint
- added TP3: +3V3, Connector_Pin:Pin_D1.3mm_L11.3mm_W2.8mm_Flat, symbol Connector:TestPoint
- added TP4: +5V, Connector_Pin:Pin_D1.3mm_L11.3mm_W2.8mm_Flat, symbol Connector:TestPoint
- added TP5: +2V5, Connector_Pin:Pin_D1.3mm_L11.3mm_W2.8mm_Flat, symbol Connector:TestPoint
Connections:
- net +2V5: now also TP5.1
- net +3V3: now also TP3.1
- net +5V: now also TP4.1
- net -0.6V: now also TP1.1
- net -5V: now also TP2.1

Commit message: 15
Parts:
- added J10, J18, J20, J21, J25: Jumper, Connector_PinHeader_2.54mm:PinHeader_1x02_P2.54mm_Vertical, symbol Connector:Conn_01x02_Pin
- added J22, J23, J24: PinHeader, Connector_PinHeader_2.54mm:PinHeader_1x02_P2.54mm_Vertical, symbol Connector:Conn_01x02_Pin
Connections:
- net +2V5: now also J21.2 (Pin_2); no longer C37.1, U7.2 (VO)
- net +3V3: now also J18.2 (Pin_2); no longer C13.1, U9.2 (VO)
- net +5V: now also J20.2 (Pin_2); no longer C22.1, U11.5 (OUT)
- net +6V: now also J22.1 (Pin_1), J22.2 (Pin_2)
- net -0.6V: now also J10.2 (Pin_2); no longer C26.1, D1.1 (K), R31.2
- net -10V: no longer R30.1
- net -5V: now also J25.2 (Pin_2); no longer C19.1, Q1.1 (E), R24.2, R26.2, U10.7 (VCC-)
- net GND: now also J23.1 (Pin_1), J23.2 (Pin_2)
- new net: C13.1, J18.1 (Pin_1), U9.2 (VO)
- new net: C19.1, J25.1 (Pin_1), Q1.1 (E), R24.2, R26.2, U10.7 (VCC-)
- new net: C22.1, J20.1 (Pin_1), U11.5 (OUT)
- new net: C26.1, D1.1 (K), J10.1 (Pin_1), R31.2
- new net: C37.1, J21.1 (Pin_1), U7.2 (VO)
- new net -6V: J24.1 (Pin_1), J24.2 (Pin_2), R30.1
Other:
- moved on the sheet: C14, C15, C16, C18, C19, C23, C24, C25, C26, D1, Q1, R23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
