File: frontend/frontend.kicad_pcb (KiCad board)
At the start: 2 copper layers, 126 x 131 mm, 176 parts, among them J1 REF_IN, J10 GND, J11 Conn_02x13_Odd_Even, J12 Conn_01x01_Socket, J13 Conn_01x01_Socket, J14 Conn_01x01_Socket, J15 Conn_01x01_Socket, J16 Conn_01x01_Socket, J17 Conn_01x01_Socket, J18 Conn_01x01_Socket, J19 A, J2 REF_S_P, J3 REF_S_N, J4 REF_GND, J5 mA, J6 V, J7 Common, J8 +6V, J9 -10V, K1 NRP26-A05D, K2 NRP26-A05D, Q1 BD136, Q2 MMBT2222A, Q3 MMBT2222A, U1 ADG722, U10 UA723, U11 NCP161, U12 MAX4208, U13 OPA2186DR, U14 ADG722, U15 74HC595, U2 ADG722, U3 OPA2186DR, U4 LM358, U5 LTC2508CDKD-32, U6 ADG722, U7 XC6206P252MR, U8 74HC595, U9 XC6206P332MR

Commit message: 10
Parts:
- U1: moved to B.Cu
- moved J11 171.4 mm to (223.5, 34.6), turned to -90 degrees
- moved U1 166.6 mm to (228.5, 86.1), turned to -90 degrees
- moved F2 91.2 mm to (152.3, 131.8)
- moved J8 67.5 mm to (178.2, 49.6), turned to 90 degrees
- moved J10 62.7 mm to (178.3, 41.4), turned to 90 degrees
- moved J9 56.9 mm to (178.2, 33.9), turned to 90 degrees
- moved H1 28.5 mm to (142.3, 137.9)
- moved H4 1.58 mm to (257.5, 138.4)
Routing:
- net REF: track 49.7 -> 48.3 mm
- net Net-(U2A-S1): vias 0 -> 1
- net Net-(U1B-S2): vias 0 -> 1
- net Net-(U1A-S1): vias 0 -> 1

Commit message: 11
Parts:
- removed J12: Conn_01x01_Socket, Connector_PinHeader_2.54mm:PinHeader_1x01_P2.54mm_Vertical
- added C56: 4u7, Capacitor_SMD:C_0805_2012Metric_Pad1.18x1.45mm_HandSolder, F.Cu at (207.8, 97.7)
- added C57: 100n, Capacitor_SMD:C_0805_2012Metric_Pad1.18x1.45mm_HandSolder, F.Cu at (194.3, 91.5)
- added C58: 4u7, Capacitor_SMD:C_0805_2012Metric_Pad1.18x1.45mm_HandSolder, F.Cu at (189.9, 102.9)
- added C59: 4u7, Capacitor_SMD:C_0805_2012Metric_Pad1.18x1.45mm_HandSolder, F.Cu at (194.8, 97.4)
- added H5: MountingHole, MountingHole:MountingHole_3.2mm_M3, F.Cu at (236.7, 56.9)
- added H6: MountingHole, MountingHole:MountingHole_3.2mm_M3, F.Cu at (245.9, 121.2)
- added H7: MountingHole, MountingHole:MountingHole_3.2mm_M3, F.Cu at (152.1, 103.1)
- added H8: MountingHole, MountingHole:MountingHole_3.2mm_M3, F.Cu at (236.7, 103.4)
- added U16: ADG722, Library:uSOIC, F.Cu at (197.2, 92.9)
- C28, C29, D2, D3, Q2, Q3, R42, R43, R54, R55, R57, U2: moved to B.Cu
- R14, R15, R2, R4, R5: value 5M/0.1% -> 2M2/0.1%
- R6: value 10k/0.1% -> 5k/0.1%
- R62: value 10 -> 47
- R7: value 100k/0.1% -> 50k/0.1%
- R8: value 1M/0.1% -> 500k/0.1%
- R9: value 20meg/0.1% -> 10meg/0.1%
- moved U2 166.6 mm to (227.8, 96.5), turned to 90 degrees
- moved U12 143.3 mm to (205.8, 102.6), turned to 90 degrees
- moved C29 141.7 mm to (225.6, 88.2), turned to 90 degrees
- moved Q2 141.7 mm to (186.3, 122.7), turned to 180 degrees
- moved C28 140.8 mm to (225.2, 98.0), turned to -90 degrees
- moved R42 140.3 mm to (209.2, 127.5), turned to -90 degrees
- moved U13 136.9 mm to (186.4, 98.4), turned to 90 degrees
- moved R43 135.3 mm to (210.0, 120.0), turned to -90 degrees
- moved H4 133.2 mm to (152.1, 56.9)
- moved R46 125.7 mm to (203.5, 115.1)
- moved R38 124.1 mm to (204.4, 96.3), turned to -90 degrees
- moved R50 123.5 mm to (199.9, 106.9)
- moved C51 123.2 mm to (105.3, 234.3)
- moved R56 123.2 mm to (96.9, 180.0)
- moved C41 123.2 mm to (92.9, 208.7)
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Connections:
- U15 pad 2: Net-(J12-Pin_1) -> /SW_CURR_10A
Routing:
- net GND: track 250.4 -> 432.3 mm, vias 25 -> 54
- net /COMMON: track 57.8 -> 180.6 mm, vias 4 -> 8
- net +5V: track 41.1 -> 158.1 mm, vias 3 -> 14
- net /SW_LOW: track 2.03 -> 103.1 mm, vias 0 -> 6
- net +1V65: track 24.0 -> 88.2 mm, vias 2 -> 8
- net /SW_RANGE10: track 0.00 -> 56.6 mm
- net /SW_RANGE100: track 0.00 -> 55.5 mm, vias 0 -> 2
- net /SW_RANGE1000: track 0.00 -> 54.9 mm
- net -0.6V: track 0.00 -> 54.4 mm, vias 0 -> 1
- net Net-(F2-Pad2): track 0.00 -> 50.5 mm
- net -5V: track 18.4 -> 68.8 mm, vias 2 -> 4
- net Net-(K2-Pad1): track 0.00 -> 40.3 mm
- net Net-(K1-Pad1): track 0.00 -> 35.2 mm, vias 0 -> 2
- net /ADC_IN+: track 27.5 -> 59.3 mm, vias 2 -> 6
- net /SW_CURR_10A: track 0.00 -> 31.0 mm, vias 0 -> 1
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- added copper zone on F.Cu, net GND
Other:
- board size 126 x 131 mm -> 114 x 131 mm

Commit message: 12
Parts:
- removed R60: 10k, Resistor_SMD:R_1206_3216Metric_Pad1.30x1.75mm_HandSolder
- added C60: 1u, Capacitor_SMD:C_0805_2012Metric_Pad1.18x1.45mm_HandSolder, F.Cu at (181.3, 97.0)
- added C61: 1u, Capacitor_SMD:C_0805_2012Metric_Pad1.18x1.45mm_HandSolder, F.Cu at (200.7, 101.4)
- added C62: 1u, Capacitor_SMD:C_0805_2012Metric_Pad1.18x1.45mm_HandSolder, F.Cu at (226.7, 68.6)
- added C63: 1u, Capacitor_SMD:C_0805_2012Metric_Pad1.18x1.45mm_HandSolder, F.Cu at (234.9, 64.6)
- U11: value NCP161 -> NCP161ASN500T1G
- moved H3 167.6 mm to (245.0, 28.0)
- moved C41 165.3 mm to (207.7, 89.8)
- moved C32 146.7 mm to (194.1, 65.6), turned to 180 degrees
- moved H2 125.6 mm to (143.0, 41.9)
- moved C51 123.4 mm to (156.5, 122.0), turned to -90 degrees
- moved R61 110.5 mm to (164.3, 28.7)
- moved C53 108.6 mm to (164.9, 32.2), turned to -90 degrees
- moved C10 107.9 mm to (150.5, 32.5), turned to -90 degrees
- moved R59 105.0 mm to (163.7, 39.2)
- moved J17 101.9 mm to (179.8, 42.6), turned to 90 degrees
- moved R35 100.6 mm to (189.5, 65.6)
- moved J18 98.7 mm to (175.7, 28.3)
- moved J16 98.1 mm to (176.0, 42.6), turned to 90 degrees
- moved C20 97.6 mm to (150.7, 105.8), turned to -90 degrees
- moved J8 97.4 mm to (144.7, 97.8)
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Connections:
- J11 pad 1: /MCLK -> /SHIFT_SRCLK
- J11 pad 10: Net-(J11-Pin_10) -> GND
- J11 pad 12: Net-(J11-Pin_10) -> GND
- J11 pad 13: /SCKA -> /SDOB
- J11 pad 14: Net-(J11-Pin_10) -> GND
- J11 pad 15: /SDOA -> /SCKB
- J11 pad 16: Net-(J11-Pin_10) -> GND
- J11 pad 17: /SCKB -> /SCKA
- J11 pad 18: Net-(J11-Pin_10) -> GND
- J11 pad 19: /SDOB -> /SDOA
- J11 pad 2: Net-(J11-Pin_10) -> GND
- J11 pad 20: Net-(J11-Pin_10) -> GND
- J11 pad 21: /SHIFT_DATA -> /DRL
- J11 pad 22: Net-(J11-Pin_10) -> GND
- J11 pad 23: /SHIFT_SRCLK -> /SYNC
- J11 pad 24: Net-(J11-Pin_10) -> GND
- J11 pad 25: /SHIFT_RCLK -> /MCLK
- J11 pad 26: /SHIFT_SRCLK -> unconnected-(J11-Pin_26-Pad26)
- J11 pad 3: /SYNC -> /SHIFT_DATA
- J11 pad 4: Net-(J11-Pin_10) -> GND
- J11 pad 5: /RDLA -> /SHIFT_RCLK
- J11 pad 6: Net-(J11-Pin_10) -> GND
- J11 pad 8: Net-(J11-Pin_10) -> GND
- J11 pad 9: /DRL -> /RDLA
- R45 pad 2: +5V -> +3V3
- R58 pad 2: +5V -> +3V3
- R59 pad 2: +5V -> +3V3
- U15 pad 1: /SW_CURR_200mA -> /SEL1
- U15 pad 15: /SW_CURR_10mA -> /SW_VOLTS_IN
- U15 pad 2: /SW_CURR_10A -> /SEL0
- U8 pad 1: /SW_RANGE100 -> /SW_CURR_RANGE
- U8 pad 15: /SW_RANGE1000 -> /SW_1V65_IN
- U8 pad 2: /SW_RANGE10 -> /SW_CURR_200mA
- U8 pad 3: /SEL0 -> /SW_CURR_10A
- U8 pad 4: /SEL1 -> /SW_RANGE10
- U8 pad 5: /SW_VOLTS_IN -> /SW_RANGE1000
- U8 pad 6: /SW_1V65_IN -> /SW_RANGE100
- U8 pad 7: /SW_CURR_RANGE -> /SW_CURR_10mA
Routing:
- net GND: track 432.3 -> 866.4 mm, vias 54 -> 130
- net -5V: track 68.8 -> 298.8 mm, vias 4 -> 8
- net +3V3: track 15.6 -> 211.5 mm, vias 0 -> 6
- net /SW_CURR_RANGE: track 2.35 -> 139.7 mm, vias 0 -> 1
- net /SW_VOLTS_IN: track 4.62 -> 113.1 mm, vias 0 -> 4
- net /SW_1V65_IN: track 6.06 -> 112.8 mm
- net /SW_LOW: track 103.1 -> 191.7 mm, vias 6 -> 10
- net /SEL1: track 4.55 -> 74.4 mm, vias 0 -> 2
- net /SEL0: track 6.37 -> 74.6 mm, vias 0 -> 2
- net -0.6V: track 54.4 -> 118.0 mm, vias 1 -> 2
- net /SW_CURR_10mA: track 16.3 -> 79.8 mm, vias 1 -> 2
- net /SW_CURR_200mA: track 14.5 -> 77.6 mm, vias 1 -> 2
- net /SW_RANGE10: track 56.6 -> 118.4 mm, vias 0 -> 1
- net /SW_CURR_10A: track 31.0 -> 92.3 mm, vias 1 -> 2
- net /SW_RANGE1000: track 54.9 -> 116.1 mm, vias 0 -> 1
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Other:
- board size 114 x 131 mm -> 114 x 122 mm
- board text added: "+6V"
- board text added: "-10V"
- board text added: "A"
- board text added: "COM"
- board text added: "GND"
- board text added: "V"
- board text added: "busy"
- board text added: "data"
- board text added: "drl"
- board text added: "mA"
- board text added: "mclk"
- board text added: "rclk"
- board text added: "rdla"
- board text added: "rdlb"
- board text added: "ref+"
- board text added: "ref_gnd"
- board text added: "ref_s_g"
- board text added: "ref_s_p"
- board text added: "scka"
- board text added: "sckb"
- board text added: "sdoa"
- board text added: "sdob"
- board text added: "srclk"
- board text added: "sync"

Commit message: 13
Parts:
- added TP1: -0.6V, Connector_Pin:Pin_D1.3mm_L11.3mm_W2.8mm_Flat, F.Cu at (153.9, 50.1)
- added TP2: -5V, Connector_Pin:Pin_D1.3mm_L11.3mm_W2.8mm_Flat, F.Cu at (165.3, 84.1)
- added TP3: +3V3, Connector_Pin:Pin_D1.3mm_L11.3mm_W2.8mm_Flat, F.Cu at (161.8, 88.2)
- added TP4: +5V, Connector_Pin:Pin_D1.3mm_L11.3mm_W2.8mm_Flat, F.Cu at (159.5, 99.9)
- added TP5: +2V5, Connector_Pin:Pin_D1.3mm_L11.3mm_W2.8mm_Flat, F.Cu at (160.7, 84.2)
- moved H3 2.06 mm to (243.0, 27.5)
- moved R15 0.77 mm to (221.0, 101.2)
- moved R14 0.77 mm to (221.0, 96.1)
- moved R28 0.41 mm to (149.0, 92.2)
Routing:
- net GND: track 866.4 -> 828.1 mm, vias 130 -> 157
- net -5V: track 298.8 -> 306.7 mm
- net -0.6V: track 118.0 -> 121.3 mm
- net +3V3: track 211.5 -> 214.2 mm
- net +2V5: track 36.6 -> 39.2 mm
- net /SW_RANGE10: track 118.4 -> 120.9 mm
- net +5V: track 216.8 -> 218.7 mm
- net +1V65: track 88.2 -> 86.3 mm
- net /SW_LOW: track 191.7 -> 192.4 mm
- added copper zone on B.Cu, net /COMMON
- added copper zone on F.Cu, net /COMMON
- added copper zone on B.Cu, net Net-(F1-Pad2)
- added copper zone on F.Cu, net Net-(F1-Pad2)
Other:
- board size 114 x 122 mm -> 111.5 x 122 mm
- board text added: "+2V5"
- board text added: "+3V3"
- board text added: "+5V"
- board text added: "-0.6V"
- board text added: "-5V"
- board text added: "14/02/2025"

Commit message: 13
Parts:
- removed C10: 100n, Capacitor_SMD:C_0805_2012Metric_Pad1.18x1.45mm_HandSolder
- removed J13, J18: Conn_01x01_Socket, Connector_PinHeader_2.54mm:PinHeader_1x01_P2.54mm_Vertical
- removed R22: 10, Resistor_SMD:R_1206_3216Metric_Pad1.30x1.75mm_HandSolder
- removed R34: 10k, Resistor_SMD:R_1206_3216Metric_Pad1.30x1.75mm_HandSolder
- removed U15: 74HC595, Package_SO:SOIC-16_3.9x9.9mm_P1.27mm
- added J12: Conn_01x01_Socket, Connector_PinHeader_2.54mm:PinHeader_1x01_P2.54mm_Vertical, F.Cu at (147.4, 33.9)
- U8: value 74HC595 -> TCA9535DBR; footprint Package_SO:SOIC-16_3.9x9.9mm_P1.27mm -> Package_SO:SSOP-24_5.3x8.2mm_P0.65mm
- moved J17 33.9 mm to (150.2, 26.0), turned to -90 degrees
- moved J16 27.6 mm to (153.9, 26.0), turned to -90 degrees
- moved J15 22.5 mm to (157.7, 25.5), turned to -90 degrees
- moved J14 18.2 mm to (161.3, 25.9), turned to -90 degrees
- moved R61 17.6 mm to (146.7, 29.5)
- moved C53 14.8 mm to (150.2, 30.4)
- moved R45 7.95 mm to (170.7, 29.6), turned to -90 degrees
- moved U8 1.46 mm to (156.0, 33.2)
- moved U2 1.17 mm to (229.0, 96.5)
- moved C28 0.83 mm to (226.0, 98.2)
- moved R2 0.15 mm to (221.6, 91.2)
Connections:
- C53 pad 1: Net-(U15-VCC) -> Net-(U8-VCC)
- J11 pad 1: /SHIFT_SRCLK -> /SDA
- J11 pad 26: unconnected-(J11-Pin_26-Pad26) -> GND
- J11 pad 3: /SHIFT_DATA -> /SCL
- J11 pad 5: /SHIFT_RCLK -> unconnected-(J11-Pin_5-Pad5)
- R61 pad 2: Net-(U15-VCC) -> Net-(U8-VCC)
- U8 pad 1: /SW_CURR_RANGE -> unconnected-(U8-~{INT}-Pad1)
- U8 pad 10: +3V3 -> /SW_RANGE100
- U8 pad 11: /SHIFT_SRCLK -> /SW_CURR_10mA
- U8 pad 12: /SHIFT_RCLK -> GND
- U8 pad 13: /SHIFT_SRCLK -> /SW_1V65_IN
- U8 pad 14: /SHIFT_DATA -> /SEL0
- U8 pad 15: /SW_1V65_IN -> /SEL1
- U8 pad 16: Net-(U8-VCC) -> /SW_VOLTS_IN
- U8 pad 2: /SW_CURR_200mA -> GND
- U8 pad 3: /SW_CURR_10A -> GND
- U8 pad 4: /SW_RANGE10 -> Net-(J12-Pin_1)
- U8 pad 5: /SW_RANGE1000 -> /SW_CURR_RANGE
- U8 pad 6: /SW_RANGE100 -> /SW_CURR_200mA
- U8 pad 7: /SW_CURR_10mA -> /SW_CURR_10A
- U8 pad 8: GND -> /SW_RANGE10
- U8 pad 9: Net-(U15-SER) -> /SW_RANGE1000
Routing:
- net /SHIFT_SRCLK: track 47.0 -> 0.00 mm, vias 2 -> 0
- net /SHIFT_RCLK: track 44.1 -> 0.00 mm
- net /SCL: track 0.00 -> 39.6 mm, vias 0 -> 1
- net +3V3: track 214.2 -> 176.0 mm, vias 6 -> 3
- net /SHIFT_DATA: track 37.3 -> 0.00 mm, vias 1 -> 0
- net /SDA: track 0.00 -> 36.3 mm, vias 0 -> 1
- net /SEL1: track 74.4 -> 87.3 mm
- net /SEL0: track 74.6 -> 87.4 mm
- net Net-(U15-SER): track 12.8 -> 0.00 mm, vias 2 -> 0
- net /SW_1V65_IN: track 112.8 -> 101.3 mm
- net Net-(J12-Pin_1): track 0.00 -> 8.89 mm
- net Net-(J13-Pin_1): track 8.07 -> 0.00 mm
- net GND: track 828.1 -> 820.8 mm
- net Net-(U15-VCC): track 5.01 -> 0.00 mm
- net Net-(J18-Pin_1): track 3.19 -> 0.00 mm
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
Commit message: 14
Parts:
- removed J10: GND, Passives:Conn-1-6x6-OD3mm
- removed J9: -10V, Passives:Conn-1-6x6-OD3mm
- J11: value Conn_02x13_Odd_Even -> 321026SG0ABK00A01
- J8: value +6V -> 2.54-2*4P, LCSC C9135; footprint Passives:Conn-1-6x6-OD3mm -> Connector_IDC:IDC-Header_2x04_P2.54mm_Vertical
- moved C12 16.1 mm to (142.5, 85.5), turned to -90 degrees
- moved C11 13.1 mm to (144.6, 85.5), turned to -90 degrees
- moved J8 12.6 mm to (150.9, 108.8)
- moved R28 11.6 mm to (147.2, 80.7), turned to -90 degrees
- moved C13 10.1 mm to (147.5, 88.7), turned to 180 degrees
- moved C20 9.35 mm to (148.0, 96.9)
- moved C21 9.35 mm to (145.9, 96.9)
- moved C22 9.35 mm to (156.4, 96.9)
- moved R29 9.35 mm to (149.8, 93.4)
- moved U11 9.35 mm to (152.6, 96.8)
- moved U9 8.73 mm to (147.7, 85.4), turned to 90 degrees
- moved TP4 3.69 mm to (163.0, 98.6)
- moved R36 3.44 mm to (149.8, 80.8), turned to -90 degrees
Connections:
- J8 pad 1: +6V -> -10V
Routing:
- net -10V: track 11.8 -> 55.1 mm
- net +6V: track 35.6 -> 56.5 mm
- net +3V3: track 176.0 -> 185.4 mm
- net +5V: track 220.7 -> 226.9 mm
Other:
- board text added: "18/02/2025 Rev A"
- board text removed: "14/02/2025"

Commit message: 15
Parts:
- added J10: Jumper, Connector_PinHeader_2.54mm:PinHeader_1x02_P2.54mm_Vertical, F.Cu at (159.7, 49.1)
- added J18: Jumper, Connector_PinHeader_2.54mm:PinHeader_1x02_P2.54mm_Vertical, F.Cu at (159.7, 92.8)
- added J20: Jumper, Connector_PinHeader_2.54mm:PinHeader_1x02_P2.54mm_Vertical, F.Cu at (159.7, 97.0)
- added J21: Jumper, Connector_PinHeader_2.54mm:PinHeader_1x02_P2.54mm_Vertical, F.Cu at (159.7, 85.2)
- added J22: PinHeader, Connector_PinHeader_2.54mm:PinHeader_1x02_P2.54mm_Vertical, F.Cu at (141.6, 93.5)
- added J23: PinHeader, Connector_PinHeader_2.54mm:PinHeader_1x02_P2.54mm_Vertical, F.Cu at (141.6, 77.1)
- added J24: PinHeader, Connector_PinHeader_2.54mm:PinHeader_1x02_P2.54mm_Vertical, F.Cu at (141.6, 100.8)
- added J25: Jumper, Connector_PinHeader_2.54mm:PinHeader_1x02_P2.54mm_Vertical, F.Cu at (159.7, 81.4)
- moved C19 10.0 mm to (154.5, 81.0), turned to 180 degrees
- moved TP1 9.74 mm to (163.0, 53.6)
- moved C23 8.19 mm to (146.3, 76.2), turned to 180 degrees
- moved TP5 7.52 mm to (155.8, 89.9)
- moved TP2 6.99 mm to (163.4, 77.3)
- moved C24 6.92 mm to (146.2, 74.0), turned to 180 degrees
- moved R24 4.76 mm to (154.0, 78.7)
- moved C35 4.10 mm to (151.4, 88.4)
- moved C36 4.10 mm to (151.4, 90.7)
- moved R31 3.24 mm to (149.7, 52.7), turned to -90 degrees
- moved C37 2.87 mm to (156.0, 85.1)
- moved U7 2.87 mm to (152.9, 84.9)
- moved R29 2.50 mm to (147.3, 93.7)
- moved TP4 2.08 mm to (163.0, 100.6)
- moved TP3 1.11 mm to (162.7, 89.0)
Connections:
- net -10V renamed -6V
- C13 pad 1: +3V3 -> Net-(J18-Pin_1)
- C19 pad 1: -5V -> Net-(J25-Pin_1)
- C22 pad 1: +5V -> Net-(J20-Pin_1)
- C26 pad 1: -0.6V -> Net-(D1-K)
- C37 pad 1: +2V5 -> Net-(J21-Pin_1)
- D1 pad 1: -0.6V -> Net-(D1-K)
- Q1 pad 1: -5V -> Net-(J25-Pin_1)
- R24 pad 2: -5V -> Net-(J25-Pin_1)
- R26 pad 2: -5V -> Net-(J25-Pin_1)
- R31 pad 2: -0.6V -> Net-(D1-K)
- U10 pad 7: -5V -> Net-(J25-Pin_1)
- U11 pad 5: +5V -> Net-(J20-Pin_1)
- U7 pad 2: +2V5 -> Net-(J21-Pin_1)
- U9 pad 2: +3V3 -> Net-(J18-Pin_1)
Routing:
- net Net-(J25-Pin_1): track 0.00 -> 43.5 mm, vias 0 -> 2
- net Net-(D1-K): track 0.00 -> 19.4 mm
- net -5V: track 308.5 -> 290.8 mm, vias 8 -> 7
- net Net-(J18-Pin_1): track 0.00 -> 16.7 mm
- net +3V3: track 185.4 -> 172.8 mm
- net +5V: track 226.9 -> 217.7 mm
- net -0.6V: track 121.3 -> 113.4 mm
- net Net-(J20-Pin_1): track 0.00 -> 6.24 mm
- net Net-(J21-Pin_1): track 0.00 -> 6.21 mm
- net -6V: track 55.1 -> 59.5 mm
- net GND: track 821.3 -> 825.6 mm, vias 157 -> 159
- net /Power/IN+: track 11.7 -> 15.1 mm
- net Net-(Q1-C): track 27.1 -> 29.9 mm
- net Net-(U7-VI): track 7.42 -> 9.77 mm
- net +6V: track 56.5 -> 55.0 mm
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Other:
- board text added: "-6V"
- board text added: "20/02/2025 Rev A"
- board text removed: "-10V"
- board text removed: "18/02/2025 Rev A"
