File: front-panel/front-panel.kicad_pcb (KiCad board)
At the start: 2 copper layers, 108.5 x 55.5 mm, 88 parts, among them J1 Conn_02x04_Odd_Even, J3 Conn_02x04_Odd_Even, U1 7-seg, 4-dig, common anode, U10 B_SAMPLES, U11 B_NLPC, U12 B, U13 TCA9535DBR, U4 7-seg, 4-dig, common anode, U5 Auto, U6 B_1V/10mA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

Commit message: 14
Parts:
- removed C15: 220u, Capacitor_Tantalum_SMD:CP_EIA-7343-31_Kemet-D
- removed TP3: TestPoint, Connector_Pin:Pin_D0.9mm_L10.0mm_W2.4mm_FlatFork
- added D6: LED, Passives:led_3mm_mid_hole, F.Cu at (214.5, 69.6)
- added R24: 470, Resistor_SMD:R_1206_3216Metric_Pad1.30x1.75mm_HandSolder, B.Cu at (213.5, 67.1)
- added REF**: 0.3mm_hole, Passives:0.3mm_hole, F.Cu at (184.0, 65.0)
- added REF**: 0.3mm_hole, Passives:0.3mm_hole, F.Cu at (235.0, 65.0)
- added REF**: 0.3mm_hole, Passives:0.3mm_hole, F.Cu at (129.5, 65.0)
- added REF**: 0.3mm_hole, Passives:0.3mm_hole, F.Cu at (182.0, 65.0)
- added REF**: 0.3mm_hole, Passives:0.3mm_hole, F.Cu at (130.5, 65.0)
- added REF**: 0.3mm_hole, Passives:0.3mm_hole, F.Cu at (236.0, 65.0)
- added REF**: 0.3mm_hole, Passives:0.3mm_hole, F.Cu at (183.0, 65.0)
- added REF**: 0.3mm_hole, Passives:0.3mm_hole, F.Cu at (131.5, 65.0)
- added REF**: 0.3mm_hole, Passives:0.3mm_hole, F.Cu at (237.0, 65.0)
- C14, R22, R23, TP1, TP13, TP14, TP2, TP4, TP5, TP6, U13: moved to B.Cu
- J1, J3: value Conn_02x04_Odd_Even -> 2.54-2*4P, LCSC C9135
- R17, R18, R19, R20, R21: value 6k8 -> 470; moved to B.Cu
- moved R16 143.1 mm to (215.0, 74.5), turned to 90 degrees
- moved R15 140.2 mm to (212.7, 74.5), turned to -90 degrees
- moved TP6 133.0 mm to (235.2, 78.9), turned to 180 degrees
- moved TP4 132.7 mm to (235.2, 75.4), turned to 180 degrees
- moved R14 132.1 mm to (205.0, 74.4), turned to 90 degrees
- moved R13 129.2 mm to (202.7, 74.4), turned to -90 degrees
- moved R12 120.6 mm to (194.5, 74.4), turned to 90 degrees
- moved R11 117.8 mm to (192.1, 74.4), turned to -90 degrees
- moved U13 115.3 mm to (174.1, 79.3)
- moved R10 110.0 mm to (184.6, 74.4), turned to 90 degrees
- moved R8 109.7 mm to (174.6, 74.4), turned to 90 degrees
- moved C13 108.6 mm to (224.1, 83.2)
- moved R9 107.4 mm to (182.2, 74.4), turned to -90 degrees
- moved R7 106.5 mm to (172.2, 74.4), turned to -90 degrees
- moved TP5 106.1 mm to (208.7, 81.4), turned to 180 degrees
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Connections:
- TP1 pad 1: Net-(U13-P05) -> Net-(U13-P10)
- TP2 pad 1: Net-(U13-P06) -> Net-(U13-P11)
- U13 pad 10: Net-(U13-P06) -> /B_100V/10A
- U13 pad 11: Net-(U13-P07) -> /LED_100V/10A
- U13 pad 13: /B_AUTO -> Net-(U13-P10)
- U13 pad 14: /B_1V/10mA -> Net-(U13-P11)
- U13 pad 15: /B_10V/200mA -> /B_1000V
- U13 pad 16: /B_100V/10A -> /LED_1000V
- U13 pad 17: /B_1000V -> /B_SAMPLES
- U13 pad 18: /B_SAMPLES -> /B_NLPC
- U13 pad 19: /B_NLPC -> /B
- U13 pad 20: /B -> /LED_HEATER
- U13 pad 4: /LED_AUTO -> /B_AUTO
- U13 pad 5: /LED_1V/10mA -> /LED_AUTO
- U13 pad 6: /LED_10V/200mA -> /B_1V/10mA
- U13 pad 7: /LED_100V/10A -> /LED_1V/10mA
- U13 pad 8: /LED_1000V -> /B_10V/200mA
- U13 pad 9: Net-(U13-P05) -> /LED_10V/200mA
Routing:
- net GNDA: track 0.00 -> 331.1 mm, vias 0 -> 1
- net +3.3VA: track 0.00 -> 210.5 mm, vias 0 -> 2
- net /INT: track 0.00 -> 79.7 mm, vias 0 -> 2
- net /SDA: track 0.00 -> 74.7 mm, vias 0 -> 3
- net /SCL: track 0.00 -> 66.7 mm, vias 0 -> 4
- net /LED_HEATER: track 0.00 -> 53.8 mm
- net /B: track 0.00 -> 46.2 mm, vias 0 -> 1
- net /B_NLPC: track 0.00 -> 36.7 mm, vias 0 -> 1
- net /LED_AUTO: track 0.00 -> 36.5 mm
- net /B_AUTO: track 0.00 -> 36.5 mm, vias 0 -> 1
- net /LED_1000V: track 0.00 -> 27.0 mm
- net /B_SAMPLES: track 0.00 -> 26.5 mm, vias 0 -> 1
- net /LED_1V/10mA: track 0.00 -> 24.8 mm
- net /B_1V/10mA: track 0.00 -> 24.6 mm, vias 0 -> 1
- net Net-(R10-Pad1): track 0.00 -> 22.2 mm, vias 0 -> 2
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- added copper zone on B.Cu, net GND
- added copper zone on F.Cu, net GND
- added copper zone on B.Cu, net GNDA
- added copper zone on F.Cu, net GNDA
Other:
- outline, holes or cut-outs redrawn
- board text added: "+"
- board text added: "18/02/25 Rev A"
- board text added: "INT"
- board text added: "SCL"
- board text added: "SDA"
