File: front-panel/front-panel.kicad_sch (KiCad schematic)
At the start: 88 parts, among them J1 Conn_02x04_Odd_Even, J3 Conn_02x04_Odd_Even, U1 7-seg, 4-dig, common anode, U10 B_SAMPLES, U11 B_NLPC, U12 B, U13 TCA9535DBR, U4 7-seg, 4-dig, common anode, U5 Auto, U6 B_1V/10mA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

Commit message: 14
Parts:
- removed C15: 220u, Capacitor_Tantalum_SMD:CP_EIA-7343-31_Kemet-D, symbol Device:C_Polarized
- removed TP3: TestPoint, Connector_Pin:Pin_D0.9mm_L10.0mm_W2.4mm_FlatFork, symbol Connector:TestPoint
- added D6: LED, Passives:led_3mm_mid_hole, symbol Device:LED
- added J2, J4: I254-2*4-G-3-B, Connector_IDC:IDC-Header_2x04_P2.54mm_Vertical, symbol Connector_Generic:Conn_02x04_Odd_Even
- added R24: 470, Resistor_SMD:R_1206_3216Metric_Pad1.30x1.75mm_HandSolder, symbol Device:R
- J1, J3: value Conn_02x04_Odd_Even -> 2.54-2*4P, LCSC C9135
- R17, R18, R19, R20, R21: value 6k8 -> 470
Connections:
- net B: now also U13.19 (P16); no longer U13.20 (P17)
- net B_1000V: now also U13.15 (P12); no longer U13.17 (P14)
- net B_100V/10A: now also U13.10 (P06); no longer U13.16 (P13)
- net B_10V/200mA: now also U13.8 (P04); no longer U13.15 (P12)
- net B_1V/10mA: now also U13.6 (P02); no longer U13.14 (P11)
- net B_AUTO: now also U13.4 (P00); no longer U13.13 (P10)
- net B_NLPC: now also U13.18 (P15); no longer U13.19 (P16)
- net B_SAMPLES: now also U13.17 (P14); no longer U13.18 (P15)
- net GNDA: now also D6.1 (K)
- net LED_1000V: now also U13.16 (P13); no longer U13.8 (P04)
- net LED_100V/10A: now also U13.11 (P07); no longer U13.7 (P03)
- net LED_10V/200mA: now also U13.9 (P05); no longer U13.6 (P02)
- net LED_1V/10mA: now also U13.7 (P03); no longer U13.5 (P01)
- net LED_AUTO: now also U13.5 (P01); no longer U13.4 (P00)
- net at TP2.1: now also U13.14 (P11); no longer U13.10 (P06)
- net at TP1.1: now also U13.13 (P10); no longer U13.9 (P05)
- new net: D6.2 (A), R24.2
- new net LED_HEATER: R24.1, U13.20 (P17)
Other:
- moved on the sheet: C1, C14, C2, D1, D2, D3, D4, R17, R18, R19, R20
