File: reference/reference.kicad_pcb (KiCad board)
At the start: 2 copper layers, 37 x 25 mm, 28 parts, among them J1 NTC, J2 HEATER, J3 Conn_01x08_Socket, Q1 IRFS4115, U1 TL431DBZ, U2 REF3433IDBVR, U3 LM358

Commit message: 4
Parts:
- removed U2: REF3433IDBVR, Package_TO_SOT_SMD:SOT-23W
- added J4: NTC, Connector_PinHeader_2.54mm:PinHeader_1x02_P2.54mm_Vertical, F.Cu at (138.8, 80.9)
- added J5: NTC, Connector_PinHeader_2.54mm:PinHeader_1x02_P2.54mm_Vertical, F.Cu at (141.3, 86.3)
- added U4: REF3433IDBVR, Package_TO_SOT_SMD:SOT-23-6, F.Cu at (146.7, 87.7)
- C11, C7, C8, R2, R5, R7, R8, R9, U3: moved to B.Cu
- moved J3 64.9 mm to (157.5, 72.1)
- moved R2 64.2 mm to (151.6, 72.5), turned to 90 degrees
- moved R6 62.0 mm to (149.4, 82.7)
- moved R1 60.4 mm to (147.6, 73.5), turned to 90 degrees
- moved R3 56.4 mm to (143.8, 72.0), turned to 180 degrees
- moved R5 56.0 mm to (142.7, 72.8), turned to -90 degrees
- moved C5 55.5 mm to (152.9, 83.4), turned to 90 degrees
- moved C3 52.9 mm to (149.1, 90.6), turned to 180 degrees
- moved R4 52.5 mm to (139.7, 73.3), turned to -90 degrees
- moved C6 51.5 mm to (148.8, 85.0), turned to 180 degrees
- moved C1 50.2 mm to (147.6, 78.1), turned to 90 degrees
- moved C4 48.3 mm to (145.0, 90.6)
- moved R8 45.8 mm to (131.1, 77.2), turned to 180 degrees
- moved R9 45.1 mm to (128.0, 74.7), turned to 180 degrees
- moved C7 44.5 mm to (146.6, 71.2), turned to 180 degrees
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Connections:
- C9 pad 2: GND2 -> Net-(J1-Pin_2)
Routing:
- net +15V: track 0.00 -> 62.2 mm, vias 0 -> 1
- net GND: track 0.00 -> 61.6 mm, vias 0 -> 4
- net GND2: track 0.00 -> 52.2 mm, vias 0 -> 2
- net Net-(U4-ENABLE): track 0.00 -> 25.9 mm, vias 0 -> 1
- net /GNDS: track 0.00 -> 25.1 mm
- net /OUTS: track 0.00 -> 23.5 mm
- net Net-(J2-Pin_1): track 0.00 -> 22.6 mm, vias 0 -> 8
- net Net-(U3A--): track 0.00 -> 14.9 mm
- net +12V: track 0.00 -> 10.1 mm
- net /OUT: track 0.00 -> 9.90 mm
- net Net-(C1-Pad2): track 0.00 -> 8.17 mm, vias 0 -> 1
- net Net-(U1-K): track 0.00 -> 7.67 mm, vias 0 -> 1
- net Net-(J1-Pin_2): track 0.00 -> 6.09 mm, vias 0 -> 1
- net Net-(J4-Pin_1): track 0.00 -> 5.39 mm
- net Net-(J4-Pin_2): track 0.00 -> 5.39 mm
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- added copper zone on B.Cu, net Net-(J2-Pin_1)
Other:
- outline, holes or cut-outs redrawn

Commit message: 16
Parts:
- R7: value ~ -> 820
- R8, R9: value ~ -> 4k7
Changed lines of the file:
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@@
 			)
 		)
-		(property "Value" "~"
+		(property "Value" "4k7"
 			(at 0 -1.82 0)
 			(layer "B.Fab")
@@
 			)
 		)
-		(property "Value" "~"
+		(property "Value" "4k7"
 			(at 0 -1.82 0)
 			(layer "B.Fab")
@@
 			)
 		)
-		(property "Value" "~"
+		(property "Value" "820"
 			(at 0 -1.82 0)
 			(layer "B.Fab")
