File: reference/reference.kicad_sch (KiCad schematic)
At the start: 14 parts, among them U1 TL431DBZ, U2 REF3433IDBVR

Commit message: ref done
Parts:
- added C10, C8: 100n, Capacitor_SMD:C_0805_2012Metric_Pad1.18x1.45mm_HandSolder, symbol Device:C
- added C11, C7: 10u, Capacitor_SMD:C_0805_2012Metric_Pad1.18x1.45mm_HandSolder, symbol Device:C
- added C9: 10n, Capacitor_SMD:C_0805_2012Metric_Pad1.18x1.45mm_HandSolder, symbol Device:C
- added J1: NTC, symbol Connector:Conn_01x02_Socket
- added J2: HEATER, symbol Connector:Conn_01x02_Socket
- added J3: Conn_01x08_Socket, symbol Connector:Conn_01x08_Socket
- added Q1: IRFS4115, Package_TO_SOT_SMD:Infineon_PG-HDSOP-10-1, symbol Transistor_FET:IRFS4115
- added R10: 470, Resistor_SMD:R_1206_3216Metric_Pad1.30x1.75mm_HandSolder, symbol Device:R
- added R7, R8, R9: ~, Resistor_SMD:R_1206_3216Metric_Pad1.30x1.75mm_HandSolder, symbol Device:R
- added U3: LM358, Package_SO:SOIC-8_3.9x4.9mm_P1.27mm, symbol Amplifier_Operational:LM358
- C2: footprint (none) -> Capacitor_Tantalum_SMD:CP_EIA-7343-31_Kemet-D
Connections:
- net +15V: now also C10.2, J2.2 (Pin_2), J3.7 (Pin_7), R7.1, R8.1, U3.8 (V+); no longer R2.1
- net GND: now also C7.1, J3.5 (Pin_5)
- net at R1.2, R3.1, R5.1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: now also C7.2
- net GNDS: now reaches U2.2 (GNDS)
- net GNDS: now also J3.1 (Pin_1)
- net OUTS: now reaches U2.5 (OUT_S)
- net OUTS: now also J3.2 (Pin_2)
- net OUT: now reaches C5.2, R6.2
- net OUT: now also J3.3 (Pin_3)
- new net: Q1.1 (G), R10.2
- new net: J2.1 (Pin_1), Q1.2 (D)
- new net: C11.2, C8.2, R8.2, R9.1, U3.2 (-)
- new net: U3.6 (-), U3.7
- new net: J1.2 (Pin_2), R7.2, U3.3 (+)
- new net: C11.1, R10.1, U3.1
- new net +12V: J3.4 (Pin_4), R2.1
- new net GND2: C10.1, C8.1, C9.1, C9.2, J1.1 (Pin_1), J3.8 (Pin_8), Q1.3 (S), R9.2, U3.4 (V-), U3.5 (+)
Other:
- moved on the sheet: C3, C4, C5, C6, R5, R6, U2

Commit message: starting pcb
Parts:
- J1, J2: footprint (none) -> Connector_PinHeader_2.54mm:PinHeader_1x02_P2.54mm_Vertical
- J3: footprint (none) -> Connector_PinHeader_2.54mm:PinHeader_1x08_P2.54mm_Vertical
- Q1: footprint Package_TO_SOT_SMD:Infineon_PG-HDSOP-10-1 -> Package_TO_SOT_SMD:TO-252-2
Changed lines of the file:
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@@
 			)
 		)
-		(property "Footprint" "Package_TO_SOT_SMD:Infineon_PG-HDSOP-10-1"
+		(property "Footprint" "Package_TO_SOT_SMD:TO-252-2"
 			(at 104.14 121.285 0)
 			(effects
@@
 			)
 		)
-		(property "Footprint" ""
+		(property "Footprint" "Connector_PinHeader_2.54mm:PinHeader_1x02_P2.54mm_Vertical"
 			(at 106.68 110.49 0)
 			(effects
@@
 			)
 		)
-		(property "Footprint" ""
+		(property "Footprint" "Connector_PinHeader_2.54mm:PinHeader_1x08_P2.54mm_Vertical"
 			(at 213.36 92.71 0)
 			(effects
@@
 			)
 		)
-		(property "Footprint" ""
+		(property "Footprint" "Connector_PinHeader_2.54mm:PinHeader_1x02_P2.54mm_Vertical"
 			(at 46.99 129.54 0)
 			(effects

Commit message: 4
Parts:
- removed U2: REF3433IDBVR, Package_TO_SOT_SMD:SOT-23W, symbol Reference_Voltage:REF3212AMDBVREP
- added J4, J5: NTC, Connector_PinHeader_2.54mm:PinHeader_1x02_P2.54mm_Vertical, symbol Connector:Conn_01x02_Socket
- added U4: REF3433IDBVR, Package_TO_SOT_SMD:SOT-23-6, symbol Reference_Voltage:REF3212AMDBVREP
Connections:
- net GND: now also U4.1 (GNDF)
- net GND2: no longer C9.2
- net GNDS: now also U4.2 (GNDS)
- net OUTS: now also U4.5 (OUT_S)
- net at C6.2, R6.1: now also U4.6 (OUT_F)
- net at C3.2, C4.2, R5.2: now also U4.3 (ENABLE), U4.4 (VIN)
- net at J1.2 (Pin_2), R7.2, U3.3 (+): now also C9.2
- new net: J4.2 (Pin_2), J5.1 (Pin_1)
- new net: J4.1 (Pin_1), J5.2 (Pin_2)

Commit message: 16
Parts:
- R7: value ~ -> 820
- R8, R9: value ~ -> 4k7
Other:
- note added: "820 at 68 deg"
Changed lines of the file:
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@@
 		)
 	)
-	(label "OUT"
-		(at 185.42 63.5 180)
-		(fields_autoplaced yes)
+	(text "820 at 68 deg"
+		(exclude_from_sim no)
+		(at 49.53 132.842 0)
 		(effects
 			(font
 				(size 1.27 1.27)
 			)
-			(justify right bottom)
-		)
-	)
-	(label "OUTS"
-		(at 148.59 66.04 180)
-		(fields_autoplaced yes)
+		)
+	)
+	(label "OUT"
+		(at 185.42 63.5 180)
 		(effects
 			(font
@@
 		)
 	)
-	(label "GNDS"
-		(at 114.3 76.2 0)
-		(fields_autoplaced yes)
+	(label "OUTS"
+		(at 148.59 66.04 180)
 		(effects
 			(font
 				(size 1.27 1.27)
 			)
-			(justify left bottom)
-		)
-	)
-	(label "OUT"
-		(at 201.93 90.17 0)
-		(fields_autoplaced yes)
+			(justify right bottom)
+		)
+	)
+	(label "GNDS"
+		(at 114.3 76.2 0)
 		(effects
 			(font
@@
 		)
 	)
-	(label "OUTS"
-		(at 201.93 87.63 0)
-		(fields_autoplaced yes)
+	(label "OUT"
+		(at 201.93 90.17 0)
 		(effects
 			(font
@@
 		)
 	)
-	(label "GNDS"
-		(at 201.93 85.09 0)
-		(fields_autoplaced yes)
+	(label "OUTS"
+		(at 201.93 87.63 0)
 		(effects
 			(font
@@
 		)
 	)
+	(label "GNDS"
+		(at 201.93 85.09 0)
+		(effects
+			(font
+				(size 1.27 1.27)
+			)
+			(justify left bottom)
+		)
+	)
 	(symbol
 		(lib_id "power:GND2")
@@
 			)
 		)
-		(property "Value" "~"
+		(property "Value" "4k7"
 			(at 38.1 111.76 0)
 			(effects
@@
 			)
 		)
-		(property "Value" "~"
+		(property "Value" "4k7"
 			(at 38.1 129.54 0)
 			(effects
@@
 			)
 		)
-		(property "Value" "~"
-			(at 54.61 111.76 0)
-			(effects
-				(font
+		(property "Value" "820"
+			(at 46.99 111.76 0)
+			(effects
+				(font

Commit message: 17
Parts:
- C11: now not fitted
Other:
- note added: "pin 1 and 2 of tl431 need to be swapped"
Changed lines of the file:
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@@
+		)
+	)
+	(text "pin 1 and 2 of tl431 need to be swapped"
+		(exclude_from_sim no)
+		(at 56.388 86.36 0)
+		(effects
+			(font
+				(size 1.27 1.27)
+			)
 		)
 	)
@@
 		(in_bom yes)
 		(on_board yes)
-		(dnp no)
+		(dnp yes)
 		(property "Reference" "C11"
 			(at 64.008 109.728 0)
